File: sens_less_blmd.brd (EAGLE design)
At the start: 100 x 80 mm, 66 parts

Commit message: 回路図を作成
Parts:
- removed CON3: (no value), user_conector:XH_4P
- removed CON4: (no value), user_conector:XH_8P
- removed IC_1: (no value), user_ic:TLP291
- removed LED2: (no value), user_leds:1608
- removed R_I1, R_I4, R_I5: (no value), user_rcl:0603X4RESISTOR
- removed R_I2, R_I3: 10k, user_rcl:1005X4RESISTOR
- removed TR1, TR2, TR3, TR4, TR5, TR6: (no value), user_tr_fet_igbt:D2PACK
- removed U$1: A4919, user_ic:TSSOP_28P_ALLEGRO_E
- removed U$10, U$11, U$12, U$13, U$8, U$9: SBR10M100P5Q, user_diode:POWERDI_5
- removed U$14, U$15: ACS711, user_ic:SOIC8
- removed U$2, U$3, U$4: TLP2105, user_ic:SOP8
- removed U$5: FDC6305, user_tr_fet_igbt:SSOT6
- added C17, C8, C9: SNB, rcl:C4532
- added D1: RB160M-30TR, user_diode:SOD_123
- added D2, D3, D4, D5, D6, D7: SBR15U30SP5, user_diode:POWERDI_5
- added D8: SMAJ22A-13-F, user_diode:DO-214AC
- added IC1: A4919, user_ic:TSSOP_28P_ALLEGRO_E
- added K1, K2, K3: TLP2105, user_ic:SOP8
- added K4: TLP291, user_ic:TLP291
- added Q1, Q2, Q3: IAUC60N04S6L045HATMA1PG-TDSON-8-57, user_tr_fet_igbt:PG-TDSON-8-57
- added Q4, Q5: AO3400A, user_tr_fet_igbt:SOT23
- added R14, R15, R19, R20, R22, R23, R24, R25, R26, R27, R28, R32, R33, R34: (no value), user_rcl:1608
- added R29: 3.3k, user_rcl:1608
- added R30: optional, user_rcl:1608
- added R31: 47k, user_rcl:1608
- added R35: OP, user_rcl:1608
- added U1, U2: ACS711, user_ic:SOIC8
- C16: value 0.1u -> 10u
- C5, C6: value (none) -> 0.1u
- CON1: device user_conector:XH_3P -> user_conector:XH_8P
- CON2: device user_conector:XH_4P -> user_conector:XH_8P
- LED1: value (none) -> RGB_LED; device user_leds:1608 -> user_leds:RGB_LED
- R13: value 10k -> (none)
- R18: value 10k -> 47k
- moved LED1 390.0 mm to (-215.9, -198.1), turned to 0 degrees
- moved CON2 307.9 mm to (-58.4, -198.1)
- moved CON1 275.5 mm to (-58.4, -190.5), turned to 0 degrees
- moved R13 206.6 mm to (-55.9, -96.5), turned to 0 degrees
- moved C2 182.5 mm to (-55.9, -81.3)
- moved C3 179.3 mm to (-55.9, -86.4)
- moved C4 176.6 mm to (-55.9, -91.4)
- moved C23 9.16 mm to (68.6, 25.4), turned to 0 degrees
Connections:
- removed net AGND: LED2.K, U$5.2, U$5.5
- removed net CURRENT_U: U$14.P$1, U$14.P$2
- removed net CURRENT_W: U$15.P$1, U$15.P$2
- removed net FAULT_O: CON1.P$2, IC_1.PIN4, R13.1
- removed net IAHI: CON4.P$3, R_I5.2
- removed net IALO: CON4.P$4, R_I5.1
- removed net IBHI: CON4.P$5, R_I4.4
- removed net IBLO: CON4.P$6, R_I4.3
- removed net ICHI: CON4.P$7, R_I4.2
- removed net ICLO: CON4.P$8, R_I4.1
- removed net N$27: R_I4.6, U$3.PIN1
- removed net N$28: R_I4.5, U$3.PIN4
- removed net N$29: R_I5.8, U$4.PIN1
- removed net N$30: R_I5.7, U$4.PIN4
- removed net N$35: CON2.P$3
- removed net N$39: CON3.P$3
- removed net U_GND: C5.2, CON2.P$1, U$14.P$5
- removed net U_OUT: CON2.P$2, U$14.P$7
- removed net U_VCC: C5.1, CON2.P$4, U$14.P$8
- removed net VCCIO: CON1.P$3, R13.2
- removed net W_GND: C6.2, CON3.P$1, U$15.P$5
- removed net W_OUT: CON3.P$2, U$15.P$7
- removed net W_VCC: C6.1, CON3.P$4, U$15.P$8
- new net MCU_AHI: CON2.P$2, R24.1
- new net MCU_ALO: CON2.P$1, R23.1
- new net MCU_BHI: CON2.P$4, R26.1
- new net MCU_BLO: CON2.P$3, R25.1
- new net MCU_CHI: CON2.P$6, R28.1
- new net MCU_CLO: CON2.P$5, R27.1
- new net MCU_FAULT: CON1.P$2, K4.PIN3, R31.2
- new net MCU_POWER: CON1.P$1, K4.PIN4, R34.1
- new net N$10: IC1.PIN19
- new net N$11: K1.PIN1, R23.2
- new net N$12: K1.PIN4, R24.2
- new net N$13: K2.PIN1, R25.2
- new net N$14: K2.PIN4, R26.2
- new net N$15: K3.PIN1, R27.2
- new net N$26: LED1.R_K, Q5.PIN3
- new net PHASE_U_OUT: U1.P$3, U1.P$4
- new net PHASE_W_OUT: U2.P$3, U2.P$4
- new net U_CURRENT: CON1.P$6, U1.P$7
- new net VREF+: C5.1, C6.1, CON1.P$4, U1.P$8, U2.P$8
- new net VREF-: C5.2, C6.2, CON1.P$5, CON1.P$7, U1.P$5, U2.P$5
- new net W_CURRENT: CON1.P$8, U2.P$7
- net AHI: now also IC1.PIN23, K1.PIN6, R22.2; no longer R_I2.8, U$1.PIN23, U$4.PIN6
- net ALO: now also IC1.PIN24, K1.PIN7, R20.2; no longer R_I2.7, U$1.PIN24, U$4.PIN7
- net BHI: now also IC1.PIN25, K2.PIN6, R19.2; no longer R_I2.6, U$1.PIN25, U$3.PIN6
- net BLO: now also IC1.PIN26, K2.PIN7, R15.2; no longer R_I2.5, U$1.PIN26, U$3.PIN7
- net CHI: now also IC1.PIN27, K3.PIN6, R14.2; no longer R_I3.8, U$1.PIN27, U$2.PIN6
- net CLO: now also IC1.PIN28, K3.PIN7, R13.2; no longer R_I3.7, U$1.PIN28, U$2.PIN7
- net FAULT: now also IC1.PIN22, Q4.PIN1, Q5.PIN1, R30.2, R35.2; no longer U$1.PIN22, U$5.1, U$5.3
- net GHA: now also IC1.PIN11; no longer U$1.PIN11
- net GHB: now also IC1.PIN7; no longer U$1.PIN7
- net GHC: now also IC1.PIN3; no longer U$1.PIN3
- net GLA: now also IC1.PIN10; no longer U$1.PIN10
- net GLB: now also IC1.PIN6; no longer U$1.PIN6
- net GLC: now also IC1.PIN2; no longer U$1.PIN2
- net GND: now also C17.2, C8.2, C9.2, D3.1, D3.2, D5.1, D5.2, D7.1, D7.2, D8.A, IC1.PIN1, Q1.5, Q1.6, Q2.5, Q2.6, Q3.5, Q3.6; no longer TR1.3, TR4.3, TR6.3, U$1.PIN1, U$10.1, U$10.2, U$13.1, U$13.2, U$9.1, U$9.2
- net GNDA: now also IC1.PAD, IC1.PAD@10, IC1.PAD@11, IC1.PAD@12, IC1.PAD@13, IC1.PAD@14, IC1.PAD@2, IC1.PAD@3, IC1.PAD@4, IC1.PAD@5, IC1.PAD@6, IC1.PAD@7, IC1.PAD@8, IC1.PAD@9, K1.PIN5, K2.PIN5, K3.PIN5, LED1.G_K, Q4.PIN2, Q5.PIN2, R13.1, R14.1, R15.1, R19.1, R20.1, R22.1, R30.1, R35.1; no longer R_I2.1, R_I2.2, R_I2.3, R_I2.4, R_I3.1, R_I3.2, U$1.PAD, U$1.PAD@2, U$1.PIN19, U$2.PIN5, U$3.PIN5, U$4.PIN5
- net GNDIO: now also CON1.P$3, CON2.P$7, CON2.P$8, K1.PIN2, K1.PIN3, K2.PIN2, K2.PIN3, K3.PIN2, K3.PIN3, LED1.B_K, R31.1; no longer CON1.P$1, CON4.P$1, IC_1.PIN3, U$2.PIN2, U$2.PIN3, U$3.PIN2, U$3.PIN3, U$4.PIN2, U$4.PIN3
- net N$1: now also Q1.1; no longer TR2.1
- net N$16: now also IC1.PIN13; no longer U$1.PIN13
- net N$17: now also IC1.PIN9; no longer U$1.PIN9
- net N$18: now also IC1.PIN5; no longer U$1.PIN5
- net N$19: now also K3.PIN4, R28.2; no longer LED1.K, U$5.4
- net N$2: now also Q1.4; no longer TR1.1
- net N$20: now also K4.PIN2, Q4.PIN3; no longer IC_1.PIN2, U$5.6
- net N$21: now also C15.1, D1.K, IC1.PIN17; no longer IC_1.PIN1, R_I1.4
- net N$22: now also K4.PIN1, R29.2; no longer LED1.A, R_I1.3
- net N$23: now also Q2.1, R3.2, R9.2; no longer LED2.A, R_I1.1
- net N$24: now also LED1.G_A, R33.2; no longer R_I4.8, U$2.PIN1
- net N$25: now also LED1.R_A, R32.2; no longer R_I4.7, U$2.PIN4
- net N$3: now also Q2.4; no longer TR4.1
- net N$4: now also LED1.B_A, R34.2; no longer R3.2, R9.2, TR3.1
- net N$5: now also Q3.1; no longer TR5.1
- net N$6: now also Q3.4; no longer TR6.1
- net N$7: now also IC1.PIN16; no longer U$1.PIN16
- net N$8: now also IC1.PIN15; no longer U$1.PIN15
- net N$9: now also IC1.PIN14; no longer U$1.PIN14
- net PHASE_U: now also D2.1, D2.2, D3.3, IC1.PIN12, Q1.2, Q1.3, U1.P$1, U1.P$2; no longer TR1.2, TR2.3, U$1.PIN12, U$14.P$3, U$14.P$4, U$8.1, U$8.2, U$9.3
- net PHASE_V: now also D4.1, D4.2, D5.3, IC1.PIN8, Q2.2, Q2.3; no longer TR3.3, TR4.2, U$1.PIN8, U$10.3, U$11.1, U$11.2
- net PHASE_W: now also D6.1, D6.2, D7.3, IC1.PIN4, Q3.2, Q3.3, U2.P$1, U2.P$2; no longer TR5.3, TR6.2, U$1.PIN4, U$12.1, U$12.2, U$13.3, U$15.P$3, U$15.P$4
- net V5: now also IC1.PIN20, K1.PIN8, K2.PIN8, K3.PIN8, R29.1, R32.1, R33.1; no longer R_I1.5, R_I1.6, R_I1.8, U$1.PIN20, U$2.PIN8, U$3.PIN8, U$4.PIN8
- net VCC: now also C17.1, C8.1, C9.1, D1.A, D2.3, D4.3, D6.3, D8.C, IC1.PIN18, Q1.7, Q1.8, Q2.7, Q2.8, Q3.7, Q3.8; no longer C15.1, TR2.2, TR3.2, TR5.2, U$1.PIN17, U$1.PIN18, U$11.3, U$12.3, U$8.3
- net VDSTH: now also IC1.PIN21; no longer U$1.PIN21

Commit message: fet側基板の完成とガーバーファイル追加
Parts:
- added U$1: XH_2P, user_conector:XH_2P
- added U$2: DCC5923L, user_heatshink:DCC5923L
- R10, R11, R12, R7, R8, R9: value 10k -> 47k
- moved R35 397.7 mm to (67.9, 45.0), turned to 180 degrees
- moved Q5 392.8 mm to (67.8, 48.2)
- moved R34 385.6 mm to (61.5, 47.0), flipped to the bottom, turned to 270 degrees
- moved R33 383.6 mm to (63.5, 47.0), flipped to the bottom, turned to 270 degrees
- moved R32 381.7 mm to (65.5, 47.0), flipped to the bottom, turned to 270 degrees
- moved LED1 374.3 mm to (64.8, 49.5), turned to 270 degrees
- moved D8 358.3 mm to (40.6, 11.4), flipped to the bottom, turned to 180 degrees
- moved D7 341.7 mm to (22.9, 53.3), flipped to the bottom, turned to 270 degrees
- moved D6 320.2 mm to (17.8, 38.1), flipped to the bottom, turned to 90 degrees
- moved D5 315.9 mm to (22.9, 36.8), flipped to the bottom, turned to 270 degrees
- moved D1 299.5 mm to (54.5, 20.4), turned to 180 degrees
- moved D4 294.4 mm to (17.8, 21.6), flipped to the bottom, turned to 90 degrees
- moved D3 290.1 mm to (22.9, 20.3), flipped to the bottom, turned to 270 degrees
- moved CON1 282.5 mm to (77.5, 57.1), turned to 180 degrees
- moved D2 268.6 mm to (17.8, 5.08), flipped to the bottom, turned to 90 degrees
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Connections:
- removed net N$10: IC1.PIN19
- net GND: now also Q1.SPAD, Q1.SPAD@1, Q2.SPAD, Q2.SPAD@1, Q3.SPAD, Q3.SPAD@1, U$1.P$2
- net GNDA: now also IC1.PIN19; no longer IC1.PAD@10, IC1.PAD@11, IC1.PAD@12, IC1.PAD@13, IC1.PAD@2, IC1.PAD@3, IC1.PAD@4, IC1.PAD@5, IC1.PAD@6, IC1.PAD@7, IC1.PAD@8, IC1.PAD@9
- net PHASE_U: now also Q1.SDPAD, Q1.SDPAD@1, Q1.SDPAD@2
- net PHASE_V: now also Q2.SDPAD, Q2.SDPAD@1, Q2.SDPAD@2
- net PHASE_W: now also Q3.SDPAD, Q3.SDPAD@1, Q3.SDPAD@2
- net VCC: now also Q1.DPAD, Q1.DPAD@1, Q2.DPAD, Q2.DPAD@1, Q3.DPAD, Q3.DPAD@1, U$1.P$1
Routing:
- net VREF-: track 0.00 -> 229.0 mm, vias 0 -> 3
- net VREF+: track 0.00 -> 215.9 mm, vias 0 -> 2
- net U_CURRENT: track 0.00 -> 153.0 mm, vias 0 -> 1
- net GNDIO: track 0.00 -> 124.9 mm
- net GNDA: track 0.00 -> 93.7 mm, vias 0 -> 30
- net PHASE_U: track 0.00 -> 86.9 mm, vias 0 -> 26
- net GND: track 0.00 -> 84.0 mm, vias 0 -> 85
- net VCC: track 0.00 -> 81.5 mm, vias 0 -> 82
- net V5: track 0.00 -> 77.3 mm, vias 0 -> 8
- net PHASE_W: track 0.00 -> 73.4 mm, vias 0 -> 31
- net PHASE_V: track 0.00 -> 71.0 mm, vias 0 -> 39
- net W_CURRENT: track 0.00 -> 61.1 mm
- net N$2: track 0.00 -> 59.5 mm, vias 0 -> 1
- net N$1: track 0.00 -> 59.2 mm, vias 0 -> 1
- net CHI: track 0.00 -> 48.7 mm, vias 0 -> 2
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- added copper zone on layer 1, net GND
- added copper zone on layer 16, net GND
- added copper zone on layer 1, net GNDA
- added copper zone on layer 16, net GNDA
- added copper zone on layer 1, net PHASE_U
- added copper zone on layer 16, net PHASE_U
- added copper zone on layer 1, net PHASE_U_OUT
- added copper zone on layer 16, net PHASE_U_OUT
- added copper zone on layer 1, net PHASE_V
- added copper zone on layer 16, net PHASE_V
- added copper zone on layer 1, net PHASE_W
- added copper zone on layer 16, net PHASE_W
- added copper zone on layer 1, net PHASE_W_OUT
- added copper zone on layer 16, net PHASE_W_OUT
- added copper zone on layer 1, net VCC
- added copper zone on layer 16, net VCC
- added copper zone on layer 1, net VREF-
- added copper zone on layer 16, net VREF-
Other:
- board size 100 x 80 mm -> 78.4 x 58.5 mm
- board text added: "0.Hayate"
- board text added: "For CoRE"
- board text added: "SLBL_MotaDora_Ver1"

Commit message: UVW結線のふっとぷりんと追加、新ガーバーファイル追加
Other:
- board text added: "U"
- board text added: "V"
- board text added: "W"
Changed lines of the file:
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@@
 <vertex x="-0.9" y="15.5"/>
 </polygon>
+<text x="12.8" y="12.1" size="2.54" layer="28" rot="MR0">U</text>
+<text x="12.7" y="28.1" size="2.54" layer="28" rot="MR0">V</text>
+<text x="12.9" y="43.3" size="2.54" layer="28" rot="MR0">W</text>
 </plain>
 <attributes>
