File: sens_less_blmd.brd (EAGLE design)
At the start: 78.4 x 58.5 mm, 81 parts, among them IC1 A4919, K1 TLP2105, K2 TLP2105, K3 TLP2105, K4 TLP291, Q1 IAUC60N04S6L045HATMA1PG-TDSON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, Q2 IAUC60N04S6L045HATMA1PG-TDSON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, Q3 IAUC60N04S6L045HATMA1PG-TDSON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, Q4 AO3400A, Q5 AO3400A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

Commit message: ガーバーファイル追加
Routing:
- net GNDA: track 93.7 -> 90.8 mm
Changed lines of the file:
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@@
 <wire x1="60.31" y1="41.29" x2="57.15" y2="44.45" width="0.3048" layer="1"/>
 <polygon width="0.3048" layer="1">
-<vertex x="55" y="13.6"/>
+<vertex x="46.5" y="13.6"/>
 <vertex x="56.8" y="13.6"/>
 <vertex x="56.8" y="8.1"/>
 <vertex x="46.5" y="8.1"/>
-<vertex x="46.5" y="12.2"/>
-<vertex x="55" y="12.2"/>
 </polygon>
 <wire x1="46.99" y1="41.91" x2="46.99" y2="44.45" width="0.508" layer="1"/>
@@
 <wire x1="60.31" y1="34.14" x2="58.34" y2="34.14" width="0.3048" layer="1"/>
 <wire x1="58.34" y1="34.14" x2="57.3572" y2="33.1572" width="0.3048" layer="1"/>
-<wire x1="53.22" y1="34.48" x2="52.92" y2="34.48" width="0.3048" layer="1"/>
-<wire x1="57.3572" y1="33.1572" x2="54.5428" y2="33.1572" width="0.3048" layer="1"/>
-<wire x1="54.5428" y1="33.1572" x2="53.22" y2="34.48" width="0.3048" layer="1"/>
+<wire x1="53.12" y1="34.48" x2="52.92" y2="34.48" width="0.3048" layer="1"/>
+<wire x1="57.3572" y1="33.1572" x2="54.4428" y2="33.1572" width="0.3048" layer="1"/>
+<wire x1="54.4428" y1="33.1572" x2="53.12" y2="34.48" width="0.3048" layer="1"/>
 </signal>
 <signal name="GHA">
@@
 <wire x1="68.3728" y1="33.3972" x2="68.3728" y2="30.78615" width="0.3048" layer="1"/>
 <wire x1="68.3728" y1="30.78615" x2="69.09375" y2="30.0652" width="0.3048" layer="1"/>
-<wire x1="69.09375" y1="30.0652" x2="70.1948" y2="30.0652" width="0.3048" layer="1"/>
-<wire x1="70.1948" y1="30.0652" x2="71.47" y2="28.79" width="0.3048" layer="1"/>
 <wire x1="63.42" y1="49.53" x2="63.42" y2="50.62" width="0.3048" layer="1"/>
 <wire x1="63.42" y1="50.62" x2="63.6" y2="50.8" width="0.3048" layer="1"/>
